Commit message: learning about xarco and launch.py

File: urdf/bebop.urdf.xacro (robot description, xacro)
@@ -14,5 +14,5 @@
   <xacro:property name="enable_laser1D" value="$(arg enable_laser1D)" />
   <!-- Instantiate bebop "mechanics" -->
-  	<xacro:include filename="$(find bebop_simulator)/urdf/bebop_base.urdf.xacro" />
+  	<xacro:include filename="$(find bebop_simulator_r2)/urdf/bebop_base.urdf.xacro" />
   	<xacro:include filename="$(find rotors_description)/urdf/component_snippets.xacro" />
   	<!-- Realistic odometry sensor with noise and bias -->

File: urdf/bebop_base.urdf.xacro (robot description, xacro)
@@ -34,5 +34,5 @@
   </xacro:property>
   <!-- Included URDF Files -->
-  <xacro:include filename="$(find bebop_simulator)/urdf/multirotor_base.urdf.xacro" />
+  <xacro:include filename="$(find bebop_simulator_r2)/urdf/multirotor_base.urdf.xacro" />
   <!-- Instantiate multirotor_base_macro once -->
   <xacro:multirotor_base_macro

File: urdf/multirotor_base.urdf.xacro (robot description, xacro)
@@ -19,5 +19,5 @@
         <origin xyz="0 0 0" rpy="0 0 0" />
         <geometry>
-          <mesh filename="package://bebop_simulator/meshes/${mesh_file}"
+          <mesh filename="package://bebop_simulator_r2/meshes/${mesh_file}"
             scale="0.001 0.001 0.001" />
           <!-- <box size="${body_width} ${body_width} ${body_height}"/> --> <!-- [m] [m] [m] -->
@@ -78,5 +78,5 @@
         <geometry>
           <!-- <cylinder length="0.005" radius="${radius_rotor}"/> --> <!-- [m] -->
-          <mesh filename="package://bebop_simulator/meshes/propeller_${direction}.dae"
+          <mesh filename="package://bebop_simulator_r2/meshes/propeller_${direction}.dae"
             scale="0.00055 0.00055 0.00055" />
           <!-- <box size="${2*radius_rotor} 0.01 0.005"/> -->

File: urdf/wind_turbine.base.urdf.xacro (robot description, xacro)
@@ -18,5 +18,5 @@
         <origin xyz="0 0 0" rpy="0 0 0" />
         <geometry>
-          <mesh filename="package://bebop_simulator/meshes/wind_turbine_base.dae"
+          <mesh filename="package://bebop_simulator_r2/meshes/wind_turbine_base.dae"
             scale="2 2 2" />
         </geometry>
@@ -25,5 +25,5 @@
         <origin xyz="0 0 0" rpy="0 0 0"/>
         <geometry>
-          <mesh filename="package://bebop_simulator/meshes/wind_turbine_base.dae"
+          <mesh filename="package://bebop_simulator_r2/meshes/wind_turbine_base.dae"
             scale="2 2 2" />
         </geometry>
@@ -45,5 +45,5 @@
         <origin xyz="0.16228 -0.00566 0.1" rpy="0 0 0" />
         <geometry>
-          <mesh filename="package://bebop_simulator/meshes/wind_turbine_rotor.dae"
+          <mesh filename="package://bebop_simulator_r2/meshes/wind_turbine_rotor.dae"
             scale="2 2 2" />
         </geometry>
@@ -52,5 +52,5 @@
         <origin xyz="0.16228 -0.00566 0.1" rpy="0 0 0"/>
         <geometry>
-          <mesh filename="package://bebop_simulator/meshes/wind_turbine_rotor.dae"
+          <mesh filename="package://bebop_simulator_r2/meshes/wind_turbine_rotor.dae"
             scale="2 2 2" />
         </geometry>

File: urdf/wind_turbine.gazebo.xacro (robot description, xacro)
@@ -15,5 +15,5 @@
   <xacro:property name="bag_file" value="wind_turbine.bag" />
   <!-- Instantiate mmuav "mechanics" -->
-  <xacro:include filename="$(find bebop_simulator)/urdf/wind_turbine.base.urdf.xacro" />
+  <xacro:include filename="$(find bebop_simulator_r2)/urdf/wind_turbine.base.urdf.xacro" />
   <xacro:include filename="$(find rotors_description)/urdf/component_snippets.xacro" />
 </robot>
